Commit message: feat(camera): 2대 구성 + udev 를 물리포트에서 serial 로 바꾼다
허브 하나에 카메라 4대를 물리면 USB 대역폭이 모자라 전송이 밀린다.
BRIO 좌·우를 빼고 cam_front(D455) + cam_stopline(C920) 2대로 줄였다.

udev 를 serial 기준으로
  예전 규칙은 물리 포트 경로(KERNELS=="1-7.3")로 잡고 있었다. 카메라를
  뽑았다 꽂거나 허브 포트를 옮기면 경로가 달라져서 심볼릭 링크가 조용히
  안 생기고, usb_cam 노드는 respawn 으로 무한 재시작만 한다 — 에러로
  멈추는 게 아니라 로그 도배로만 나타나서 알아채기 어렵다.
  ATTRS{serial} 은 어느 허브 어느 포트에 꽂아도 안 변한다.

  tools/cam_setup.sh 는 "BRIO 2대는 VID:PID 가 같아서 물리 포트가 유일한
  해법" 이라고 적고 있는데 이건 by-id 경로 기준으로만 맞다. serial 은
  개체마다 다르다 (BRIO 좌 BF5AC6D2 / 우 EBA07419). README 에 적어뒀다.

  udev/99-gigacha-cameras.rules 가 원본이고 /etc 로 install 해서 쓴다.

cone 기본값 false
  cone.launch 는 /cam_left, /cam_right 를 먹는데 그 두 대가 없다.
  true 로 두면 object_detector 2개가 영영 안 오는 이미지를 기다리며
  GPU 메모리만 잡는다. launch 헤더에도 경고를 달았다.

cameras.launch
  cam_left / cam_right 노드를 뺐다 (respawn=true 라 없는 /dev 를 물고
  무한 재시작하고 있었다). d455 는 기본 꺼짐 유지 — 주행 스택에서는
  traversability_live.launch 가 D455 를 열고, D455 는 한 프로세스만
  열 수 있다. 그쪽도 이제 cam_front 이름을 쓰므로 접두어가 같다.

urdf 는 left_pitch 의 "14,0" 오타를 "14.0" 으로 고쳤다 (쉼표라 xacro 가
그대로 문자열로 읽는다).

Co-Authored-By: Claude Opus 5 (1M context) <noreply@anthropic.com>
Claude-Session: https://claude.ai/code/session_01SpwGSHWf1pYfXLcQ8qmd7Z

File: urdf/gigacha_sensors.urdf.xacro (robot description, xacro)
@@ -65,5 +65,5 @@
   <xacro:property name="left_z"      value="0.300"/>   <!-- 지면 0.450 -->
   <xacro:property name="left_roll"   value="0.0"/>
-  <xacro:property name="left_pitch"  value="14,0"/>     <!-- 노면을 내려보면 양수 -->
+  <xacro:property name="left_pitch"  value="14.0"/>     <!-- 노면을 내려보면 양수 -->
   <xacro:property name="left_yaw"    value="90.0"/>     <!-- 좌측을 보면 양수 -->
   <!-- ── BRIO 우측 ──────────────────────────────────────────────────── -->

Commit message: feat(perception): 지면 좌표 발행 + 뎁스 + 미션 게이트, TensorRT 엔진 지원
제어팀에 넘기는 좌표계와 인지 노드 기동 방식을 정리한 09-15~09-19 작업.

지면 투영 / 좌표 발행
  - ground_markers.py 신설. /detect/* 2D 검출을 base_link x, y 로 바꿔
    /perception/obstacle 로 내는 유일한 발행자. 트래킹 + 시간 투표.
  - obstacle_detector 는 /perception/obstacle 발행을 넘기고 /detect/obstacle 만 낸다.
    obstacle 엔진을 두 번 올리지 않으려고 추론 결과를 그대로 내보낸다.
  - utils/ground.py, utils/obstacle_ground.py. 카메라 기하는 URDF 실측 한 곳에서.

S자 코스
  - obstacle_depth.py + utils/obstacle_depth.py: D455 정렬 뎁스를 박스별로
    지면 투영과 대조해 맞을 때만 쓰고, 틀어지면 지면 점으로 대체 → /obstacles/camera.
  - utils/s_course.py: 첫 T870 좌/우를 다수결로 커밋 → /perception/s_course/right.

미션 게이트
  - utils/mission_gate.py. 제어 GRM 의 /global_active_map + /global_nearest_idx 로
    해당 미션 구간에서만 추론한다. 신호등 15 m 전부터, 장애물은 S코스·돌발·신호차량만.
    GRM 토픽이 2초 넘게 없으면 항상 켜진다(단독 시험).

TensorRT
  - object_detector / obstacle_detector 가 .engine 로드. .to() 는 .pt 일 때만,
    task="detect" 명시, imgsz 를 predict 에 전달(엔진은 export imgsz 고정).
    엔진인데 CUDA 가 없으면 조용히 CPU 로 가지 않고 죽는다.
  - tools/export_trt.py, weights/*.engine.json 은 gitignore.

교정 / 튜닝
  - classes.yaml obstacle 라벨 순서를 학습 data.yaml(ASCII 정렬)에 맞춤.
    어긋나 있어서 좌우 지시가 뒤바뀔 수 있었다 (class_map 대조가 잡음).
  - URDF 카메라 pitch 실측 반영, 정지선 tau 를 실측 기하로 재계산 [20,45,80]→[15,30,55].
  - traffic_light ROI 를 상단 절반(0,0,1280,480)으로. 지평선 아래 오검출 제거.
  - viz_hz 를 루프 주기와 맞춤. 5 로 두면 격자가 어긋나 실측 4 Hz 대로 떨어졌다.
  - detections 토픽을 /perception/*/detections → /detect/* 로 (내부 배선과 분리).

검증 도구
  - tools/verify_{ground_markers,obstacle_depth,s_course,mission_gate}.py
  - tools/bag_obstacle_depth.py, src/bev_viz.py, docs/OBSTACLE_CAMERA_TOPIC.md

Co-Authored-By: Claude Opus 5 (1M context) <noreply@anthropic.com>

File: urdf/gigacha_sensors.urdf.xacro (robot description, xacro)
@@ -56,5 +56,7 @@
   <xacro:property name="front_z"     value="0.850"/>   <!-- 지면 1.000 -->
   <xacro:property name="front_roll"  value="0.0"/>
-  <xacro:property name="front_pitch" value="-1.0"/>     <!-- 현장에서 확정, 위를 보면 음수 -->
+  <!-- 2026-09-17: -1.0 -> -2.75. songdo_full_20260916_005609.bag 노면 뎁스 평면 실측 (높이는 0.974 로
+       나왔지만 줄자 1.000 을 유지 — 이 조합이 콘 뎁스와 지면 투영 거리 차 중앙값 -0.02 m 로 가장 맞았다) -->
+  <xacro:property name="front_pitch" value="-2.75"/>     <!-- 위를 보면 음수 -->
   <xacro:property name="front_yaw"   value="0.0"/>
   <!-- ── C920 (전방 하향 / 정지선) ──────────────────────────────────── -->
